File: eaglecad/rev2/VSCard_v2.brd (EAGLE design)
At the start: 130.2 x 73.3 mm, 51 parts, among them IC1 74LS244N, IC2 74LS08N, IC8 74LS244N, J2 RCA, J3 RCA, J4 RCA, J5 RCA, Q1 10.738635mhz, Q2 2N2222, U1 TMS4416, U11 SN76489, U2 TMS9118, U3 TMS4416, U4 SN76489

Commit message: schematic updates
Parts:
- removed C11: 10uf, rcl:E3,5-10
- added C4: 10uf, resistor:E2,5-5
- added R8: (no value), resistor:RTRIM64W
- moved R1 16.3 mm to (121.3, 51.4)
- moved R3 8.84 mm to (117.5, 26.0), turned to 270 degrees
- moved R5 7.01 mm to (125.1, 36.8), turned to 180 degrees
- moved R7 4.55 mm to (115.9, 57.1), turned to 0 degrees
- moved D1 3.84 mm to (116.8, 61.9)
- moved C5 0.63 mm to (108.0, 59.1)
Connections:
- new net N$4: J3.PIN, J3.SWITCH, R8.2
- net COMVID-OUT: now also R8.3; no longer J3.PIN, J3.SWITCH
- net GND: now also C4.-; no longer C11.-
- net VCC: now also C4.+; no longer C11.+
Routing:
- net N$94: track 66.7 -> 97.8 mm, vias 0 -> 1
- net N$4: track 0.00 -> 24.3 mm
- net N$24: track 27.1 -> 11.2 mm
- net N$64: track 114.4 -> 110.1 mm
- net COMVID-OUT: track 20.1 -> 23.2 mm
- net VCC: track 298.8 -> 297.0 mm
- net N$20: track 4.13 -> 5.42 mm
- net N$1: track 11.5 -> 12.3 mm
- net VOLTAGE-IN: track 105.6 -> 105.0 mm
Other:
- board text added: "Lum"
