File: eaglecad/rev2/VSCard_v2.sch (EAGLE design)
At the start: 51 parts, among them IC1 74LS244N, IC2 74LS08N, IC8 74LS244N, J2 RCA, J3 RCA, J4 RCA, J5 RCA, Q1 10.738635mhz, Q2 2N2222, U1 TMS4416, U11 SN76489, U2 TMS9118, U3 TMS4416, U4 SN76489

Commit message: schematic updates
Parts:
- removed C11: 10uf, rcl:CPOL-USE3.5-10
- added C4: 10uf, resistor:CPOL-USE2.5-5
- added R8: (no value), resistor:R-TRIMM64W
Connections:
- new net N$4: J3.PIN, J3.SWITCH, R8.S
- net COMVID-OUT: now also R8.E; no longer J3.PIN, J3.SWITCH
- net GND: now also C4.-; no longer C11.-
- net VCC: now also C4.+; no longer C11.+
Changed lines of the file:
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@@
 <part name="GND22" library="supply1" library_urn="urn:adsk.eagle:library:371" deviceset="GND" device=""/>
 <part name="P+11" library="supply1" library_urn="urn:adsk.eagle:library:371" deviceset="VCC" device=""/>
-<part name="C11" library="rcl" library_urn="urn:adsk.eagle:library:334" deviceset="CPOL-US" device="E3.5-10" package3d_urn="urn:adsk.eagle:package:23351/1" value="10uf"/>
 <part name="C5" library="rcl" library_urn="urn:adsk.eagle:library:334" deviceset="CPOL-US" device="E3.5-10" package3d_urn="urn:adsk.eagle:package:23351/1" value="100uf"/>
 <part name="GND25" library="supply1" library_urn="urn:adsk.eagle:library:371" deviceset="GND" device=""/>
@@
 <part name="JP1" library="jumper" library_urn="urn:adsk.eagle:library:252" deviceset="JP1E" device="" package3d_urn="urn:adsk.eagle:package:15455/1" value="INT_JP"/>
 <part name="S1" library="switch" library_urn="urn:adsk.eagle:library:380" deviceset="320-916" device="" package3d_urn="urn:adsk.eagle:package:27678/1"/>
+<part name="C4" library="resistor" library_urn="urn:adsk.eagle:library:348" deviceset="CPOL-US" device="E2.5-5" package3d_urn="urn:adsk.eagle:package:25841/1" value="10uf"/>
+<part name="R8" library="resistor" library_urn="urn:adsk.eagle:library:348" deviceset="R-TRIMM" device="64W" package3d_urn="urn:adsk.eagle:package:26055/1"/>
 </parts>
 <sheets>
@@
 <instance part="GND22" gate="1" x="160.02" y="60.96"/>
 <instance part="P+11" gate="VCC" x="251.46" y="76.2"/>
-<instance part="C11" gate="G$1" x="414.02" y="33.02"/>
 <instance part="C5" gate="G$1" x="388.62" y="33.02"/>
 <instance part="GND25" gate="1" x="17.78" y="88.9" rot="R90"/>
@@
 <instance part="JP1" gate="A" x="33.02" y="53.34"/>
 <instance part="S1" gate="1" x="368.3" y="40.64" rot="R270"/>
+<instance part="C4" gate="G$1" x="414.02" y="33.02"/>
+<instance part="R8" gate="G$1" x="309.88" y="2.54" rot="R90"/>
 </instances>
 <busses>
@@
 <pinref part="GND7" gate="1" pin="GND"/>
 <wire x1="414.02" y1="27.94" x2="414.02" y2="20.32" width="0.1524" layer="91"/>
-<pinref part="C11" gate="G$1" pin="-"/>
 <pinref part="IC8" gate="P" pin="GND"/>
 <wire x1="414.02" y1="20.32" x2="424.18" y2="20.32" width="0.1524" layer="91"/>
@@
 <wire x1="434.34" y1="25.4" x2="429.26" y2="25.4" width="0.1524" layer="91"/>
 <junction x="429.26" y="25.4"/>
+<pinref part="C4" gate="G$1" pin="-"/>
 </segment>
 <segment>
@@
 <wire x1="414.02" y1="53.34" x2="414.02" y2="35.56" width="0.1524" layer="91"/>
 <wire x1="406.4" y1="35.56" x2="414.02" y2="35.56" width="0.1524" layer="91"/>
-<pinref part="C11" gate="G$1" pin="+"/>
-<junction x="414.02" y="35.56"/>
 <pinref part="REG1" gate="G$1" pin="VOUT"/>
 <pinref part="IC8" gate="P" pin="VCC"/>
@@
 <wire x1="419.1" y1="58.42" x2="419.1" y2="53.34" width="0.1524" layer="91"/>
 <junction x="419.1" y="53.34"/>
+<pinref part="C4" gate="G$1" pin="+"/>
+<junction x="414.02" y="35.56"/>
 </segment>
 <segment>
@@
 <segment>
 <pinref part="Q2" gate="1" pin="E"/>
-<wire x1="294.64" y1="12.7" x2="309.88" y2="12.7" width="0.1524" layer="91"/>
 <pinref part="R3" gate="G$1" pin="1"/>
 <wire x1="294.64" y1="12.7" x2="294.64" y2="7.62" width="0.1524" layer="91"/>
+<wire x1="302.26" y1="2.54" x2="302.26" y2="12.7" width="0.1524" layer="91"/>
+<wire x1="302.26" y1="12.7" x2="294.64" y2="12.7" width="0.1524" layer="91"/>
 <junction x="294.64" y="12.7"/>
-<pinref part="J3" gate="G$1" pin="PIN"/>
-<pinref part="J3" gate="G$1" pin="SWITCH"/>
-<wire x1="309.88" y1="15.24" x2="309.88" y2="12.7" width="0.1524" layer="91"/>
-<junction x="309.88" y="12.7"/>
+<pinref part="R8" gate="G$1" pin="E"/>
+<wire x1="304.8" y1="2.54" x2="302.26" y2="2.54" width="0.1524" layer="91"/>
 </segment>
 </net>
@@
 </segment>
 </net>
+<net name="N$4" class="0">
+<segment>
+<pinref part="J3" gate="G$1" pin="PIN"/>
+<pinref part="J3" gate="G$1" pin="SWITCH"/>
+<wire x1="309.88" y1="15.24" x2="309.88" y2="12.7" width="0.1524" layer="91"/>
+<wire x1="309.88" y1="12.7" x2="309.88" y2="7.62" width="0.1524" layer="91"/>
+<junction x="309.88" y="12.7"/>
+<pinref part="R8" gate="G$1" pin="S"/>
+</segment>
+</net>
